File: HyperDAC.kicad_pcb (KiCad board)
At the start: 2 copper layers, 60 x 80 mm, 181 parts, among them J1 USB4085, J10 Conn_01x02, J11 DAC_MAIN_OUT, J12 ADC_1_IN, J13 ADC_2_IN, J2 POW, J3 POW, J4 STDC14, J5 VCP, J6 MINISWD, J7 Conn_01x10, J8 Conn_01x10, J9 Conn_01x02, SW1 BTN, SW2 BTN, SW3 BTN, SW4 BTN, U1 STM32H7B0VBT6, U10 OPA2387DGKR, U11 TS5A3159DBV, U12 TS5A3159DBV, U13 TS5A3159DBV, U14 AD8656, U15 AD8656, U2 ADP7142AUJZ-3.3, U3 ADP7142AUJZ-3.3, U4 M24256-BR, U5 ADR4525BRZ, U6 AD8656, U7 AD8656, U8 TS5A3159DBV, U9 TS5A3159DBV, Y1 12MHz

Commit message: routing in progress
Parts:
- removed SW4: BTN, Button_Switch_SMD:SW_SPST_B3SL-1022P
- moved C3 127.2 mm to (97.8, 75.1), turned to 45 degrees
- moved C2 125.2 mm to (104.7, 74.7), turned to 45 degrees
- moved R1 121.8 mm to (105.7, 75.7), turned to 45 degrees
- moved C4 120.6 mm to (106.7, 76.7), turned to 45 degrees
- moved C13 117.6 mm to (96.2, 114.0), turned to 180 degrees
- moved C45 113.9 mm to (124.8, 84.0)
- moved D2 111.0 mm to (92.0, 120.0), turned to 90 degrees
- moved D4 105.7 mm to (86.0, 120.0), turned to 90 degrees
- moved C43 105.3 mm to (124.8, 82.2)
- moved C15 104.0 mm to (96.0, 108.0), turned to 180 degrees
- moved SW2 103.4 mm to (82.0, 113.0), turned to 90 degrees
- moved SW3 102.8 mm to (90.0, 113.0), turned to 90 degrees
- moved C42 101.9 mm to (124.6, 77.0), turned to 180 degrees
- moved J3 100.0 mm to (79.5, 95.5)
- moved D1 93.9 mm to (106.0, 119.7), turned to 90 degrees
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Other:
- outline, holes or cut-outs redrawn

Commit message: Production ready
Parts:
- added C67: 100n 50V, Capacitor_SMD:C_0603_1608Metric_Pad1.08x0.95mm_HandSolder, F.Cu at (91.4, 58.8)
- added R54: 1Meg 1%, Resistor_SMD:R_0603_1608Metric_Pad0.98x0.95mm_HandSolder, B.Cu at (120.7, 52.6)
- added R55: 1Meg 1%, Resistor_SMD:R_0603_1608Metric_Pad0.98x0.95mm_HandSolder, B.Cu at (98.7, 52.5)
- added REF**: Fiducial_1mm_Mask2mm, Fiducial:Fiducial_1mm_Mask2mm, F.Cu at (71.5, 76.0)
- added REF**: Fiducial_1mm_Mask2mm, Fiducial:Fiducial_1mm_Mask2mm, F.Cu at (121.5, 120.5)
- added REF**: Fiducial_1mm_Mask2mm, Fiducial:Fiducial_1mm_Mask2mm, F.Cu at (111.0, 43.5)
- added REF**: Fiducial_1mm_Mask2mm, Fiducial:Fiducial_1mm_Mask2mm, B.Cu at (71.5, 76.0)
- added REF**: Fiducial_1mm_Mask2mm, Fiducial:Fiducial_1mm_Mask2mm, B.Cu at (121.5, 120.5)
- added REF**: Fiducial_1mm_Mask2mm, Fiducial:Fiducial_1mm_Mask2mm, B.Cu at (111.0, 43.5)
- added kibuzzard-6440F6E9: G***, kibuzzard-6440F6E9, F.Cu at (81.2, 80.0)
- added kibuzzard-6440F782: G***, kibuzzard-6440F782, F.Cu at (79.5, 93.5)
- added kibuzzard-6440F78E: G***, kibuzzard-6440F78E, F.Cu at (82.0, 93.5)
- added kibuzzard-6440F78E: G***, kibuzzard-6440F78E, F.Cu at (89.3, 93.5)
- added kibuzzard-6440F79B: G***, kibuzzard-6440F79B, F.Cu at (86.7, 93.5)
- added kibuzzard-64412532: G***, kibuzzard-64412532, B.Cu at (122.0, 44.0)
- added kibuzzard-64412543: G***, kibuzzard-64412543, B.Cu at (100.0, 44.0)
- added kibuzzard-6441254C: G***, kibuzzard-6441254C, B.Cu at (78.0, 44.0)
- C10, C12, C23, C24, C25, C26, C27, C28, C29, C3, C30, C31, C32, C33, C34, C63, C64, C65, C66, C8, FB1, FB3, FB4, FB5, FB6, R2, R23, R24, R25, R26, R3, R41, R42, R43, R44, R50, R51, R52, R53, TP1, TP10, TP11, TP12, TP13, TP14, TP15, TP16, TP17, TP2, TP3, TP4, TP5, TP6, TP7, TP8, TP9, U2, U3: moved to B.Cu
- moved R31 118.0 mm to (71.3, 65.9), turned to -90 degrees
- moved TP10 112.0 mm to (94.3, 67.6), turned to 180 degrees
- moved R46 110.6 mm to (75.3, 71.6), turned to 180 degrees
- moved TP15 110.5 mm to (81.1, 60.6), turned to 180 degrees
- moved TP3 109.6 mm to (79.5, 75.9), turned to 180 degrees
- moved C46 109.4 mm to (81.7, 68.9), turned to 90 degrees
- moved R20 109.4 mm to (80.8, 61.0)
- moved C41 107.5 mm to (73.9, 65.8), turned to -90 degrees
- moved R7 104.8 mm to (81.1, 87.1)
- moved TP12 104.4 mm to (89.4, 76.3), turned to 180 degrees
- moved TP5 102.5 mm to (84.7, 86.7), turned to 180 degrees
- moved R45 102.3 mm to (88.0, 56.7), turned to 90 degrees
- moved C52 102.2 mm to (75.3, 68.7), turned to 180 degrees
- moved R38 102.0 mm to (92.7, 64.3), turned to 90 degrees
- moved R13 101.3 mm to (81.8, 119.9), turned to -90 degrees
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Connections:
- net Net-(J7-Pad2) renamed /PE0
- net Net-(J7-Pad3) renamed /PE1
- net Net-(J7-Pad4) renamed /PE2
- net Net-(J7-Pad5) renamed /PE3
- net Net-(J7-Pad6) renamed /PE4
- net Net-(J7-Pad7) renamed /PE5
- net Net-(J7-Pad8) renamed /PE6
- net Net-(J7-Pad9) renamed /PE7
- net Net-(J8-Pad2) renamed /PE8
- net Net-(J8-Pad3) renamed /PE9
- net Net-(J8-Pad4) renamed /PE10
- net Net-(J8-Pad5) renamed /PE11
- net Net-(J8-Pad6) renamed /PE12
- net Net-(J8-Pad7) renamed /PE13
- net Net-(J8-Pad8) renamed /PE14
- net Net-(J8-Pad9) renamed /PE15
- J6 pad 2: unconnected-(J6-Pad2) -> /SWDIO
- R50 pad 2: /ADC1_INP16 -> /ADC2_INP1
- R51 pad 2: /ADC1_INN16 -> /ADC2_INN1
- R52 pad 2: /ADC2_INP1 -> /ADC1_INP16
- R53 pad 2: /ADC2_INN1 -> /ADC1_INN16
- TP10 pad 1: /ADC2_INN1 -> Net-(C62-Pad1)
- TP6 pad 1: /ADC1_INP16 -> Net-(C56-Pad2)
- TP8 pad 1: /ADC1_INN16 -> Net-(C61-Pad1)
- TP9 pad 1: /ADC2_INP1 -> Net-(C57-Pad2)
- U1 pad 54: /BTN3 -> unconnected-(U1-Pad54)
- U13 pad 2: (no net) -> GND
- U13 pad 5: (no net) -> +3.3VA
- U6 pad 1: Net-(C41-Pad1) -> Net-(C39-Pad1)
- U6 pad 2: Net-(C41-Pad2) -> Net-(C39-Pad2)
- U6 pad 3: /analog/REF_1.25 -> Net-(R21-Pad2)
- U7 pad 1: Net-(C39-Pad1) -> Net-(C41-Pad1)
- U7 pad 2: Net-(C39-Pad2) -> Net-(C41-Pad2)
- U7 pad 3: Net-(R21-Pad2) -> /analog/REF_1.25
Routing:
- net GND: track 0.00 -> 286.8 mm, vias 0 -> 81
- net +3.3VA: track 0.00 -> 190.4 mm, vias 0 -> 9
- net +3V3: track 0.00 -> 147.7 mm, vias 0 -> 10
- net /analog/REF_1.25: track 0.00 -> 95.5 mm, vias 0 -> 7
- net /ADC_REF_COUPLING: track 0.00 -> 85.9 mm, vias 0 -> 4
- net VBUS: track 0.00 -> 78.3 mm, vias 0 -> 2
- net /NRST: track 0.00 -> 59.5 mm, vias 0 -> 2
- net /analog/ADC1_INPUT: track 0.00 -> 52.8 mm, vias 0 -> 4
- net /LED1: track 0.00 -> 48.5 mm, vias 0 -> 3
- net /ADC_SUM_DAC_COUPLING: track 0.00 -> 47.0 mm, vias 0 -> 3
- net /VCP_RX: track 0.00 -> 44.1 mm, vias 0 -> 1
- net /LED2: track 0.00 -> 42.1 mm, vias 0 -> 2
- net /ADC_DAC_COUPLING: track 0.00 -> 41.6 mm, vias 0 -> 3
- net /VCP_TX: track 0.00 -> 40.8 mm, vias 0 -> 1
- net /SWO: track 0.00 -> 39.5 mm, vias 0 -> 2
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- added copper zone on F.Cu, net /REF_2.5
- added copper zone on F.Cu, net /analog/REF_1.25
- added copper zone on B.Cu, net GND
- added copper zone on F.Cu, net GND
- added copper zone on In1.Cu, net GND
- added copper zone on In2.Cu, net GND
Other:
- copper layers 2 -> 4
- board text added: "0"
- board text added: "1"
- board text added: "1.25"
- board text added: "2"
- board text added: "2.5"
- board text added: "3"
- board text added: "4"
- board text added: "April 2023"
- board text added: "Designed by: Jakub Mnich"
- board text added: "G"
- board text added: "GND"
- board text added: "PE1"
- board text added: "PE10"
- board text added: "PE11"
- board text added: "PE12"
- board text added: "PE13"
- board text added: "PE14"
- board text added: "PE15"
- board text added: "PE2"
- board text added: "PE3"
- board text added: "PE4"
- board text added: "PE5"
- board text added: "PE6"
- board text added: "PE7"
- board text added: "PE8"
- board text added: "PE9"
- board text added: "Rx"
- board text added: "Tx"
- board text added: "VCP"
