File: HyperDAC.kicad_sch (KiCad schematic)
At the start: 39 parts

Commit message: sch done
Parts:
- removed C? (x3): 1u 50V, Capacitor_SMD:C_0603_1608Metric_Pad1.08x0.95mm_HandSolder, symbol Device:C_Small
- removed C? (x3): 100n 50V, Capacitor_SMD:C_0603_1608Metric_Pad1.08x0.95mm_HandSolder, symbol Device:C_Small
- removed R? (x2): 10k 0.1%, Resistor_SMD:R_0603_1608Metric_Pad0.98x0.95mm_HandSolder, symbol Device:R_Small
- removed U?: ADR4525BRZ, Package_SO:SOIC-8_3.9x4.9mm_P1.27mm, symbol Reference_Voltage:ADR4520
- removed U? (x3): AD8656, Package_SO:MSOP-8_3x3mm_P0.65mm, symbol Amplifier_Operational:AD8620
- added C13: 10n 50V, Capacitor_SMD:C_0603_1608Metric, symbol Device:C_Small
- added C14, C19, C27, C28, C29, C30: 10u 25V, Capacitor_SMD:C_0805_2012Metric_Pad1.18x1.45mm_HandSolder, symbol Device:C_Small
- added C15, C22, C23, C24, C33, C34: 100n 50V, Capacitor_SMD:C_0603_1608Metric_Pad1.08x0.95mm_HandSolder, symbol Device:C_Small
- added C16: 220u 10V, Capacitor_SMD:CP_Elec_6.3x7.7, symbol Device:C_Polarized_Small
- added C25, C26, C31, C32: 1u 50V, Capacitor_SMD:C_0603_1608Metric_Pad1.08x0.95mm_HandSolder, symbol Device:C_Small
- added C35: 100n 50V, Capacitor_SMD:C_0603_1608Metric, symbol Device:C_Small
- added D1, D2, D3, D4: LED G, LED_SMD:LED_0603_1608Metric_Pad1.05x0.95mm_HandSolder, symbol Device:LED_Small
- added FB2, FB3, FB4, FB5, FB6: 100R 100MHz, Inductor_SMD:L_0805_2012Metric_Pad1.05x1.20mm_HandSolder, symbol Device:FerriteBead_Small
- added J1: USB4085, GCT_USB4085:USB_C_Receptacle_GCT_USB4085, symbol Connector:USB_C_Receptacle_USB2.0
- added J2, J3: POW, Connector_PinHeader_2.54mm:PinHeader_2x04_P2.54mm_Vertical, symbol Connector_Generic:Conn_02x04_Odd_Even
- added J5: VCP, Connector_PinHeader_2.54mm:PinHeader_1x02_P2.54mm_Vertical, symbol Connector_Generic:Conn_01x02
- added J6: MINISWD, 10pin_1.27_socket:10pin_1.27_socket, symbol Connector:Conn_ARM_JTAG_SWD_10
- added J7, J8: Conn_01x10, Connector_PinHeader_2.54mm:PinHeader_1x10_P2.54mm_Vertical, symbol Connector_Generic:Conn_01x10
- added R11, R12, R13, R14: 1k 1%, Resistor_SMD:R_0603_1608Metric_Pad0.98x0.95mm_HandSolder, symbol Device:R_Small
- added R15, R16: 2k2 1%, Resistor_SMD:R_0603_1608Metric, symbol Device:R_Small
- added R2, R3: 5k1 1%, Resistor_SMD:R_0603_1608Metric_Pad0.98x0.95mm_HandSolder, symbol Device:R_Small
- added R4, R7, R9: 47k 1%, Resistor_SMD:R_0603_1608Metric_Pad0.98x0.95mm_HandSolder, symbol Device:R_Small
- added R5, R6: 22R 1%, Resistor_SMD:R_0603_1608Metric_Pad0.98x0.95mm_HandSolder, symbol Device:R_Small
- added R8: 1k5 1%, Resistor_SMD:R_0603_1608Metric_Pad0.98x0.95mm_HandSolder, symbol Device:R_Small
- added SW1, SW2, SW3, SW4: BTN, Button_Switch_SMD:SW_SPST_B3SL-1022P, symbol Switch:SW_Push
- added U2, U3: ADP7142AUJZ-3.3, Package_TO_SOT_SMD:TSOT-23-5, symbol Regulator_Linear:ADP7142AUJZ-3.3
- added U4: M24256-BR, Package_SO:SOIC-8_3.9x4.9mm_P1.27mm, symbol M24256-BR:M24256-BR
- gave numbers to parts that had none: 22
Connections:
- net +3.3VA: now also C32.1, C34.1, FB6.2
- net +3V3: now also J4.3 (VCC), C19.1, C31.1, C33.1, C35.2, FB5.2, J3.1 (Pin_1), J3.3 (Pin_3), J3.5 (Pin_5), J3.7 (Pin_7), J6.1 (VTref), R15.1, R16.1, U4.8 (VCC)
- net GND: now also J4.11 (GNDDetect), J4.5 (GND), J4.7 (GND), C13.2, C14.2, C15.2, C16.2, C19.2, C22.2, C23.2, C24.2, C25.2, C26.2, C27.2, C28.2, C29.2, C30.2, C31.2, C32.2, C33.2, C34.2, C35.1, D1.1 (K), D2.1 (K), D3.1 (K), D4.1 (K), J1.A1 (GND), J1.A12 (GND), J1.B1 (GND), J1.B12 (GND), J1.S1 (SHIELD), J2.2 (Pin_2), J2.4 (Pin_4), J2.6 (Pin_6), J2.8 (Pin_8), J3.2 (Pin_2), J3.4 (Pin_4), J3.6 (Pin_6), J3.8 (Pin_8), J6.3 (GND), J6.5 (GND), J6.9 (GNDDetect), J7.1 (Pin_1), J7.10 (Pin_10), J8.1 (Pin_1), J8.10 (Pin_10), R2.1, R3.1, R4.1, R7.1, R9.1, SW1.2, SW2.2, SW3.2, SW4.2, U2.2 (GND), U3.2 (GND), U4.1 (E0), U4.2 (E1), U4.3 (E2), U4.4 (VSS)
- net LED2: now reaches U1.46 (PB10)
- net LED2: now also R13.2
- net LED3: now reaches U1.47 (PB11)
- net LED3: now also R14.2
- net BTN1: now reaches U1.52 (PB13)
- net BTN1: now also SW2.1
- net BTN2: now reaches U1.53 (PB14)
- net BTN2: now also SW3.1
- net BTN3: now reaches U1.54 (PB15)
- net BTN3: now also SW4.1
- net SWO: now reaches U1.89 (PB3)
- net SWO: now also J4.8 (JTDO/SWO), J6.6 (SWO/TDO)
- net SCL: now reaches U1.92 (PB6)
- net SCL: now also R16.2, U4.6 (SCL)
- net SDA: now reaches U1.93 (PB7)
- net SDA: now also R15.2, U4.5 (SDA)
- net LED1: now reaches U1.96 (PB9)
- net LED1: now also R12.2
- net ADC2_INN1: now reaches U1.17 (PC2_C)
- net ADC2_INP1: now reaches U1.18 (PC3_C)
- net VCP_RX: now reaches U1.78 (PC10)
- net VCP_RX: now also J4.13 (VCP_RX), J5.1 (Pin_1)
- net VCP_TX: now reaches U1.79 (PC11)
- net VCP_TX: now also J4.14 (VCP_TX), J5.2 (Pin_2)
- net ADC_DAC_COUPLING: now reaches U1.58 (PD11)
- net ADC_DAC_COUPLING: now also R4.2
- net ADC_SUM_DAC_COUPLING: now reaches U1.59 (PD12)
- net ADC_SUM_DAC_COUPLING: now also R7.2
- net ADC_REF_COUPLING: now reaches U1.60 (PD13)
- net ADC_REF_COUPLING: now also R9.2
- net at U1.1 (PE2): now also J7.4 (Pin_4)
- net at U1.2 (PE3): now also J7.5 (Pin_5)
- net at U1.3 (PE4): now also J7.6 (Pin_6)
- net at U1.37 (PE7): now also J7.9 (Pin_9)
- net at U1.38 (PE8): now also J8.2 (Pin_2)
- net at U1.39 (PE9): now also J8.3 (Pin_3)
- net at U1.4 (PE5): now also J7.7 (Pin_7)
- net at U1.40 (PE10): now also J8.4 (Pin_4)
- net at U1.41 (PE11): now also J8.5 (Pin_5)
- net at U1.42 (PE12): now also J8.6 (Pin_6)
- net at U1.43 (PE13): now also J8.7 (Pin_7)
- net at U1.44 (PE14): now also J8.8 (Pin_8)
- net at U1.45 (PE15): now also J8.9 (Pin_9)
- net at U1.5 (PE6): now also J7.8 (Pin_8)
- net at U1.97 (PE0): now also J7.2 (Pin_2)
- net at U1.98 (PE1): now also J7.3 (Pin_3)
- net ADC1_INP16: now reaches U1.22 (PA0)
- net ADC1_INN16: now reaches U1.23 (PA1)
- net DAC1_OUT1: now reaches U1.28 (PA4)
- net DAC1_OUT2: now reaches U1.29 (PA5)
- net USB_DP_PULL: now reaches U1.69 (PA10)
- net USB_DP_PULL: now also R8.2
- net USB_DM: now reaches U1.70 (PA11)
- net USB_DM: now also R5.2
- net USB_DP: now reaches U1.71 (PA12)
- net USB_DP: now also R6.2, R8.1
- net SWDIO: now reaches U1.72 (PA13)
- net SWDIO: now also J4.4 (JTMS/SWDIO), J6.7 (KEY)
- net SWCLK: now reaches U1.76 (PA14)
- net SWCLK: now also J4.6 (JCLK/SWCLK), J6.4 (SWDCLK/TCK)
- net NRST: now reaches U1.14 (NRST)
- net NRST: now also J4.12 (~{RST}), C22.1, J6.10 (~{RESET}), SW1.1
- new net: C13.1, FB2.2, J1.A4 (VBUS), J1.A9 (VBUS), J1.B4 (VBUS), J1.B9 (VBUS)
- new net: C29.1, FB5.1, U2.5 (VOUT)
- new net: D1.2 (A), R11.1
- new net: C30.1, FB6.1, U3.5 (VOUT)
- new net: C27.1, FB3.1, U2.1 (VIN), U2.3 (EN)
- new net: D2.2 (A), R12.1
- new net: C28.1, FB4.1, U3.1 (VIN), U3.3 (EN)
- new net: J1.A6 (D+), J1.B6 (D+), R6.1
- new net: D4.2 (A), R14.1
- new net: D3.2 (A), R13.1
- new net: J1.A5 (CC1), R2.2
- new net: J1.A7 (D-), J1.B7 (D-), R5.1
- new net: J1.B5 (CC2), R3.2
- new net VBUS: C14.1, C15.1, C16.1, C23.1, C24.1, C25.1, C26.1, FB2.1, FB3.2, FB4.2, J2.1 (Pin_1), J2.3 (Pin_3), J2.5 (Pin_5), J2.7 (Pin_7), R11.2
- no-connect marks 4 -> 47
Other:
- added sheet analog (analog.kicad_sch)
- note added: "Memory address: mem. array: 0x50 (0b1010000) ID page: 0x58 (0b1011000)"
- moved on the sheet: C1, C10, C11, C12, C17, C18, C2, C20, C21, C3, C4, C5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

Commit message: routing in progress
Parts:
- removed SW4: BTN, Button_Switch_SMD:SW_SPST_B3SL-1022P, symbol Switch:SW_Push
Connections:
- net BTN3: no longer names the net of U1.54 (PB15)
- no-connect marks 47 -> 48
Changed lines of the file:
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@@
   (junction (at 186.69 214.63) (diameter 0) (color 0 0 0 0)
   )
-  (junction (at 224.79 130.81) (diameter 0) (color 0 0 0 0)
-  )
   (junction (at 74.93 53.34) (diameter 0) (color 0 0 0 0)
   )
@@
   (junction (at 49.53 33.02) (diameter 0) (color 0 0 0 0)
   )
+  (no_connect (at 391.16 101.6))
   (no_connect (at 361.95 203.2))
   (no_connect (at 391.16 124.46))
@@
     (stroke (width 0) (type default) (color 0 0 0 0))
   )
-  (wire (pts (xy 222.25 130.81) (xy 224.79 130.81))
-    (stroke (width 0) (type default) (color 0 0 0 0))
-  )
   (wire (pts (xy 134.62 57.15) (xy 137.16 57.15))
     (stroke (width 0) (type default) (color 0 0 0 0))
@@
     (stroke (width 0) (type default) (color 0 0 0 0))
   )
-  (wire (pts (xy 204.47 130.81) (xy 212.09 130.81))
-    (stroke (width 0) (type default) (color 0 0 0 0))
-  )
   (wire (pts (xy 80.01 142.24) (xy 80.01 147.32))
     (stroke (width 0) (type default) (color 0 0 0 0))
@@
     (stroke (width 0) (type default) (color 0 0 0 0))
   )
-  (wire (pts (xy 224.79 130.81) (xy 224.79 118.11))
-    (stroke (width 0) (type default) (color 0 0 0 0))
-  )
   (wire (pts (xy 233.68 214.63) (xy 238.76 214.63))
     (stroke (width 0) (type default) (color 0 0 0 0))
@@
     (stroke (width 0) (type default) (color 0 0 0 0))
   )
-  (wire (pts (xy 224.79 134.62) (xy 224.79 130.81))
+  (wire (pts (xy 224.79 118.11) (xy 224.79 134.62))
     (stroke (width 0) (type default) (color 0 0 0 0))
   )
@@
     (stroke (width 0) (type default) (color 0 0 0 0))
   )
-  (wire (pts (xy 377.19 101.6) (xy 391.16 101.6))
-    (stroke (width 0) (type default) (color 0 0 0 0))
-  )
   (wire (pts (xy 124.46 214.63) (xy 134.62 214.63))
     (stroke (width 0) (type default) (color 0 0 0 0))
@@
     (effects (font (size 1.27 1.27)) (justify left bottom))
   )
-  (label "BTN3" (at 377.19 101.6 0)
-    (effects (font (size 1.27 1.27)) (justify left bottom))
-  )
   (label "DAC1_OUT1" (at 71.12 134.62 0)
     (effects (font (size 1.27 1.27)) (justify left bottom))
@@
     (effects (font (size 1.27 1.27)) (justify left bottom))
   )
-  (label "BTN3" (at 204.47 130.81 0)
-    (effects (font (size 1.27 1.27)) (justify left bottom))
-  )
   (label "SWDIO" (at 231.14 43.815 0)
     (effects (font (size 1.27 1.27)) (justify left bottom))
@@
     (pin "2")
   )
-  (symbol (lib_id "Switch:SW_Push") (at 217.17 130.81 0) (unit 1)
-    (in_bom yes) (on_board yes) (fields_autoplaced)
-    (property "Reference" "SW4" (id 0) (at 217.17 123.19 0))
-    (property "Value" "BTN" (id 1) (at 217.17 125.73 0))
-    (property "Footprint" "Button_Switch_SMD:SW_SPST_B3SL-1022P" (id 2) (at 217.17 125.73 0)
-      (effects (font (size 1.27 1.27)) hide)
-    )
-    (property "Datasheet" "~" (id 3) (at 217.17 125.73 0)
-      (effects (font (size 1.27 1.27)) hide)
-    )
-    (property "jlc" "C318884" (id 4) (at 217.17 130.81 0)
-      (effects (font (size 1.27 1.27)) hide)
-    )
-    (pin "1")
-    (pin "2")
-  )
   (symbol (lib_id "Device:C_Small") (at 82.55 72.39 0) (unit 1)
     (in_bom yes) (on_board yes)
@@
       (reference "SW3") (unit 1) (value "BTN") (footprint "Button_Switch_SMD:SW_SPST_B3SL-1022P")
     )
-    (path "/522058e8-9bf7-414f-bc3c-5215dcfe6796"
-      (reference "SW4") (unit 1) (value "BTN") (footprint "Button_Switch_SMD:SW_SPST_B3SL-1022P")
-    )
     (path "/2f559fa4-9c89-4d72-abbf-4fd4dc8371ba/7259e8b8-5fd6-4d31-a662-858774ca6399"

Commit message: Production ready
Connections:
- net SWDIO: now also J6.2 (SWDIO/TMS); no longer J6.7 (KEY)
- net PE0: now reaches J7.2 (Pin_2), U1.97 (PE0)
- net PE1: now reaches J7.3 (Pin_3), U1.98 (PE1)
- net PE2: now reaches J7.4 (Pin_4), U1.1 (PE2)
- net PE3: now reaches J7.5 (Pin_5), U1.2 (PE3)
- net PE4: now reaches J7.6 (Pin_6), U1.3 (PE4)
- net PE5: now reaches J7.7 (Pin_7), U1.4 (PE5)
- net PE6: now reaches J7.8 (Pin_8), U1.5 (PE6)
- net PE7: now reaches J7.9 (Pin_9), U1.37 (PE7)
- net PE8: now reaches J8.2 (Pin_2), U1.38 (PE8)
- net PE9: now reaches J8.3 (Pin_3), U1.39 (PE9)
- net PE10: now reaches J8.4 (Pin_4), U1.40 (PE10)
- net PE11: now reaches J8.5 (Pin_5), U1.41 (PE11)
- net PE12: now reaches J8.6 (Pin_6), U1.42 (PE12)
- net PE13: now reaches J8.7 (Pin_7), U1.43 (PE13)
- net PE14: now reaches J8.8 (Pin_8), U1.44 (PE14)
- net PE15: now reaches J8.9 (Pin_9), U1.45 (PE15)
Other:
- moved on the sheet: J4, J5, J6
