File: analog.kicad_sch (KiCad schematic)
At the start: 101 parts, among them J10 Conn_01x02, J11 DAC_MAIN_OUT, J12 ADC_1_IN, J13 ADC_2_IN, J9 Conn_01x02, U10 OPA2387DGKR, U11 TS5A3159DBV, U12 TS5A3159DBV, U13 TS5A3159DBV, U14 AD8656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

Commit message: Production ready
Parts:
- added C67: 100n 50V, Capacitor_SMD:C_0603_1608Metric_Pad1.08x0.95mm_HandSolder, symbol Device:C_Small
- added R54, R55: 1Meg 1%, Resistor_SMD:R_0603_1608Metric_Pad0.98x0.95mm_HandSolder, symbol Device:R_Small
- added unit 2 of U13
- renumbered U7 to U6, U6 to U7
Connections:
- net +3.3VA: now also C67.1, U13.5 (V+)
- net ADC1_INN16: now also R53.2; no longer R51.2, TP8.1
- net ADC1_INP16: now also R52.2; no longer R50.2, TP6.1
- net ADC2_INN1: now also R51.2; no longer R53.2, TP10.1
- net ADC2_INP1: now also R50.2; no longer R52.2, TP9.1
- net GND: now also C67.2, R54.1, R55.1, U13.2 (GND)
- net at C61.1, R39.1, R42.1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: now also TP8.1
- net at C57.2, R37.2, R43.1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: now also TP9.1
- net at J12.1 (In), R48.2: now also R54.2
- net at C56.2, R35.2, R41.1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: now also TP6.1
- net at J13.1 (In), R49.2: now also R55.2
- net at C62.1, R40.1, R44.1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: now also TP10.1
Other:
- moved on the sheet: R47, R48, R49, TP10, TP15, TP16, TP17, TP6, TP8, TP9
